File: untitled.brd (EAGLE design)
At the start: 100.5 x 80.4 mm, 197 parts

Commit message: Changed LED signal names to match pinmap.txt
Connections:
- net N$2 renamed HE2-G
- net N$3 renamed HE1-G
- net N$4 renamed BEDFET-G
- net N$8 renamed FET1-G
- net N$88 renamed FET2-G
- net PA2 renamed LED4
- net PC1 renamed LED5
- net PC19 renamed USBDET
- removed net LED0: R50.2, U$8.P$107
- removed net PA0: R54.2, U$8.P$109
- new net LED3: R49.1, U$8.P$45
- new net LED9: R53.2, U$8.P$110
- net LED1: now also R47.1, U$8.P$47; no longer R51.2, U$8.P$108
- net LED2: now also R48.1, U$8.P$46; no longer R53.2, U$8.P$110
- net LED6: now also R54.2, U$8.P$109; no longer R47.1, U$8.P$47
- net LED7: now also R50.2, U$8.P$107; no longer R48.1, U$8.P$46
- net LED8: now also R51.2, U$8.P$108; no longer R49.1, U$8.P$45
Routing:
- net LED3: track 0.00 -> 20.0 mm, vias 0 -> 2
- net LED8: track 20.0 -> 3.96 mm, vias 2 -> 0
- net LED6: track 17.9 -> 3.02 mm, vias 2 -> 0
- net LED7: track 16.5 -> 1.98 mm, vias 2 -> 0
- net LED1: track 3.96 -> 17.9 mm, vias 0 -> 2
- net LED2: track 4.26 -> 16.5 mm, vias 0 -> 2
- net LED9: track 0.00 -> 4.26 mm
- net PA0: track 3.02 -> 0.00 mm
- net LED0: track 1.98 -> 0.00 mm
Changed lines of the file:
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@@
 <via x="86.7" y="10.6" extent="1-16" drill="0.3"/>
 </signal>
-<signal name="N$2">
+<signal name="HE2-G">
 <contactref element="U$8" pad="P$103"/>
 <contactref element="R61" pad="2"/>
@@
 <via x="60.025" y="21.575" extent="1-16" drill="0.3"/>
 </signal>
-<signal name="N$3">
+<signal name="HE1-G">
 <contactref element="U$8" pad="P$102"/>
 <contactref element="R62" pad="2"/>
@@
 <via x="59.15" y="22.125" extent="1-16" drill="0.3"/>
 </signal>
-<signal name="N$4">
+<signal name="BEDFET-G">
 <contactref element="U$8" pad="P$101"/>
 <contactref element="R58" pad="2"/>
@@
 <wire x1="39.625" y1="36.65" x2="40.85" y2="36.65" width="0.2032" layer="1"/>
 </signal>
-<signal name="N$8">
+<signal name="FET1-G">
 <contactref element="U$8" pad="P$106"/>
 <contactref element="R60" pad="2"/>
@@
 </polygon>
 </signal>
-<signal name="N$88">
+<signal name="FET2-G">
 <contactref element="U$8" pad="P$105"/>
 <contactref element="R59" pad="1"/>
@@
 <wire x1="84.95" y1="47.875" x2="86.15" y2="47.875" width="0.4064" layer="1"/>
 </signal>
-<signal name="LED8">
+<signal name="LED3">
 <contactref element="U$8" pad="P$45"/>
 <contactref element="R49" pad="1"/>
@@
 <via x="65" y="45.05" extent="1-16" drill="0.3"/>
 </signal>
-<signal name="LED7">
+<signal name="LED2">
 <contactref element="U$8" pad="P$46"/>
 <contactref element="R48" pad="1"/>
@@
 <via x="64.05" y="44.7" extent="1-16" drill="0.3"/>
 </signal>
-<signal name="LED6">
+<signal name="LED1">
 <contactref element="U$8" pad="P$47"/>
 <contactref element="R47" pad="1"/>
@@
 <via x="60.975" y="45.85" extent="1-16" drill="0.3"/>
 </signal>
-<signal name="LED0">
+<signal name="LED7">
 <contactref element="R50" pad="2"/>
 <contactref element="U$8" pad="P$107"/>
@@
 <wire x1="56.525" y1="18.95" x2="56.1" y2="18.775" width="0.2032" layer="1"/>
 </signal>
-<signal name="LED1">
+<signal name="LED8">
 <contactref element="U$8" pad="P$108"/>
 <contactref element="R51" pad="2"/>
@@
 <wire x1="54.475" y1="17.175" x2="55.175" y2="17.875" width="0.2032" layer="1"/>
 </signal>
-<signal name="LED2">
+<signal name="LED9">
 <contactref element="R53" pad="2"/>
 <contactref element="U$8" pad="P$110"/>
@@
 <wire x1="82.675" y1="14.275" x2="75.75" y2="16.85" width="0" layer="19" extent="1-16"/>
 </signal>
-<signal name="PA0">
+<signal name="LED6">
 <contactref element="R54" pad="2"/>
 <contactref element="U$8" pad="P$109"/>
@@
 <wire x1="57.825" y1="15.4" x2="59.75" y2="16.85" width="0" layer="19" extent="1-16"/>
 </signal>
-<signal name="PA2">
+<signal name="LED4">
 <contactref element="R52" pad="2"/>
 <contactref element="U$8" pad="P$113"/>
@@
 <wire x1="93.605" y1="5.305" x2="79.25" y2="20.85" width="0" layer="19" extent="1-16"/>
 </signal>
-<signal name="PC1">
+<signal name="LED5">
 <contactref element="R55" pad="2"/>
 <contactref element="U$8" pad="P$112"/>
@@
 <wire x1="55.13" y1="28.095" x2="57.75" y2="30.85" width="0" layer="19" extent="1-16"/>
 </signal>
-<signal name="PC19">
-<contactref element="R38" pad="2"/>
-<contactref element="R37" pad="1"/>
+<signal name="USBDET">
 <contactref element="U$8" pad="P$32"/>
-<wire x1="88.675" y1="36.225" x2="88.525" y2="35.025" width="0.254" layer="1"/>
-<wire x1="88.65" y1="36.15" x2="88.675" y2="36.225" width="0.2032" layer="1"/>
 <wire x1="86.025" y1="36.15" x2="88.65" y2="36.15" width="0.2032" layer="1"/>
 <wire x1="82.5" y1="36.15" x2="86.025" y2="36.15" width="0.2032" layer="16"/>
@@
 <via x="86.025" y="36.15" extent="1-16" drill="0.3"/>
 <via x="80.65" y="34.5" extent="1-16" drill="0.3"/>
-<wire x1="88.525" y1="35.025" x2="88.675" y2="36.225" width="0" layer="19" extent="1-16"/>
-<wire x1="88.675" y1="36.225" x2="79.25" y2="34.35" width="0" layer="19" extent="1-16"/>
+<contactref element="R38" pad="2"/>
+<contactref element="R37" pad="1"/>
+<wire x1="88.675" y1="36.225" x2="88.525" y2="35.025" width="0.254" layer="1"/>
+<wire x1="88.65" y1="36.15" x2="88.675" y2="36.225" width="0" layer="19" extent="1-1"/>
 </signal>
 <signal name="PC21">
